Commit message: v9 canopy: single-feature caps, snaps, screw-in pin + repo cleanup
Body (part_body.py):
- head/rump rebuilt as ONE tall loft (dropped dome+skirt+keel-chamfer that read
  as two stacked lobes) -> each cap a single smooth feature; belly leg relief
- spine stiffener rib under the crown strips (T-beam) tying head-trunk-rump
- snaps: lateral detent nubs + alignment posts + central-wall pegs into the
  spine rib + collar grip rings on the head/rump caps (wall pockets/cups to match)

Frame (framemin.py):
- retention nubs, alignment posts + central-wall pegs (removeSplitter-per-fuse
  to survive the truss-window seam)
- printed screw-in splay pin: O7.8 pilot + P2.0 thread mating the collar bore +
  slotted O13 head -> sm3sg90_pin (print x4)

Horn: ARM is now the canonical (no-suffix) horn for coxa + legs
(coxablock CANON=arm + _sfx flip; legflat_v9 arm-only export).

Assembly (dog14.py): bakes in the real pin (framemin PIN), pegs, and the
snap-on body canopy.

Cleanup: pruned v3-v8 legs, old body/frame, stale exporters/views (~96 files to
a local attic); canonical print set = 11 watertight STLs; URDF regenerated on
the arm meshes; gitignore servos/ (208MB local reference).

Co-Authored-By: Claude Opus 4.8 <noreply@anthropic.com>

File: control/robodog.urdf (robot description, URDF)
Before this commit: robot robodog, 13 links, 12 joints
Links:
- link base_link: mass 0.05742 -> 3.563629e-02; geometry collision mesh filename=C:/ultrafish/robodog/stl/sm3sg90_v9_frame.stl scale=0.001 0.001 0.001; visual mesh filename=C:/ultrafish/robodog/stl/sm3sg90_v9_frame.stl scale=0.001 0.001 0.001
- link fl_coxa: mass 0.00315 -> 1.055894e-02; geometry collision mesh filename=C:/ultrafish/robodog/stl/sm3sg90_coxa.stl scale=0.001 0.001 0.001; collision mesh filename=C:/ultrafish/robodog/stl/sm3sg90_coxa_cover.stl scale=0.001 0.001 0.001
- link fl_femur: mass 0.01653 -> 6.769587e-03; geometry collision mesh filename=C:/ultrafish/robodog/stl/sm3sg90_v9_femur.stl scale=0.001 0.001 0.001; visual mesh filename=C:/ultrafish/robodog/stl/sm3sg90_v9_femur.stl scale=0.001 0.001 0.001
- link fl_tibia: mass 0.01454 -> 2.671392e-03; geometry collision mesh filename=C:/ultrafish/robodog/stl/sm3sg90_v9_tibia.stl scale=0.001 0.001 0.001; visual mesh filename=C:/ultrafish/robodog/stl/sm3sg90_v9_tibia.stl scale=0.001 0.001 0.001
- link fr_coxa: mass 0.00315 -> 1.055894e-02; geometry collision mesh filename=C:/ultrafish/robodog/stl/sm3sg90_coxa_cover_mir.stl scale=0.001 0.001 0.001; collision mesh filename=C:/ultrafish/robodog/stl/sm3sg90_coxa_mir.stl scale=0.001 0.001 0.001
- link fr_femur: mass 0.01653 -> 6.769908e-03; geometry collision mesh filename=C:/ultrafish/robodog/stl/sm3sg90_v9_femur_mir.stl scale=0.001 0.001 0.001; visual mesh filename=C:/ultrafish/robodog/stl/sm3sg90_v9_femur_mir.stl scale=0.001 0.001 0.001
- link fr_tibia: mass 0.01454 -> 2.672339e-03; geometry collision mesh filename=C:/ultrafish/robodog/stl/sm3sg90_v9_tibia_mir.stl scale=0.001 0.001 0.001; visual mesh filename=C:/ultrafish/robodog/stl/sm3sg90_v9_tibia_mir.stl scale=0.001 0.001 0.001
- link rl_coxa: mass 0.00315 -> 1.055894e-02; geometry collision mesh filename=C:/ultrafish/robodog/stl/sm3sg90_coxa_cover_mir.stl scale=0.001 0.001 0.001; collision mesh filename=C:/ultrafish/robodog/stl/sm3sg90_coxa_mir.stl scale=0.001 0.001 0.001
- link rl_femur: mass 0.01653 -> 6.769908e-03; geometry collision mesh filename=C:/ultrafish/robodog/stl/sm3sg90_v9_femur_mir.stl scale=0.001 0.001 0.001; visual mesh filename=C:/ultrafish/robodog/stl/sm3sg90_v9_femur_mir.stl scale=0.001 0.001 0.001
- link rl_tibia: mass 0.01454 -> 2.672339e-03; geometry collision mesh filename=C:/ultrafish/robodog/stl/sm3sg90_v9_tibia_mir.stl scale=0.001 0.001 0.001; visual mesh filename=C:/ultrafish/robodog/stl/sm3sg90_v9_tibia_mir.stl scale=0.001 0.001 0.001
- link rr_coxa: mass 0.00315 -> 1.055894e-02; geometry collision mesh filename=C:/ultrafish/robodog/stl/sm3sg90_coxa.stl scale=0.001 0.001 0.001; collision mesh filename=C:/ultrafish/robodog/stl/sm3sg90_coxa_cover.stl scale=0.001 0.001 0.001
- link rr_femur: mass 0.01653 -> 6.769587e-03; geometry collision mesh filename=C:/ultrafish/robodog/stl/sm3sg90_v9_femur.stl scale=0.001 0.001 0.001; visual mesh filename=C:/ultrafish/robodog/stl/sm3sg90_v9_femur.stl scale=0.001 0.001 0.001
- link rr_tibia: mass 0.01454 -> 2.671392e-03; geometry collision mesh filename=C:/ultrafish/robodog/stl/sm3sg90_v9_tibia.stl scale=0.001 0.001 0.001; visual mesh filename=C:/ultrafish/robodog/stl/sm3sg90_v9_tibia.stl scale=0.001 0.001 0.001
Joints:
- joint fl_knee: limit lower=-2.1817 upper=2.1817 effort=2.0 velocity=8.0 -> lower=-1.2217 upper=1.2217 effort=2.0 velocity=8.0; origin xyz=0.000000 0.000000 -0.085000 -> xyz=0.000000 0.000000 -0.070000
- joint fl_pitch: limit lower=-1.7453 upper=1.7453 effort=2.0 velocity=8.0 -> lower=-1.5708 upper=1.5708 effort=2.0 velocity=8.0; origin xyz=0.100000 -0.027200 -0.002000 -> xyz=0.082650 -0.027200 0.000000
- joint fl_splay: limit lower=-0.9599 upper=0.9599 effort=2.0 velocity=8.0 -> lower=-0.7854 upper=0.7854 effort=2.0 velocity=8.0; origin xyz=0.000000 0.027200 0.012000 -> xyz=0.000000 0.027200 0.010398
- joint fr_knee: limit lower=-2.1817 upper=2.1817 effort=2.0 velocity=8.0 -> lower=-1.2217 upper=1.2217 effort=2.0 velocity=8.0; origin xyz=0.000000 0.000000 -0.085000 -> xyz=0.000000 0.000000 -0.070000
- joint fr_pitch: limit lower=-1.7453 upper=1.7453 effort=2.0 velocity=8.0 -> lower=-1.5708 upper=1.5708 effort=2.0 velocity=8.0; origin xyz=0.100000 0.027200 -0.002000 -> xyz=0.082650 0.027200 0.000000
- joint fr_splay: limit lower=-0.9599 upper=0.9599 effort=2.0 velocity=8.0 -> lower=-0.7854 upper=0.7854 effort=2.0 velocity=8.0; origin xyz=0.000000 -0.027200 0.012000 -> xyz=0.000000 -0.027200 0.010398
- joint rl_knee: limit lower=-2.1817 upper=2.1817 effort=2.0 velocity=8.0 -> lower=-1.2217 upper=1.2217 effort=2.0 velocity=8.0; origin xyz=0.000000 0.000000 -0.085000 -> xyz=0.000000 0.000000 -0.070000
- joint rl_pitch: limit lower=-1.7453 upper=1.7453 effort=2.0 velocity=8.0 -> lower=-1.5708 upper=1.5708 effort=2.0 velocity=8.0; origin xyz=-0.100000 -0.027200 -0.002000 -> xyz=-0.082650 -0.027200 0.000000
- joint rl_splay: limit lower=-0.9599 upper=0.9599 effort=2.0 velocity=8.0 -> lower=-0.7854 upper=0.7854 effort=2.0 velocity=8.0; origin xyz=0.000000 0.027200 0.012000 -> xyz=0.000000 0.027200 0.010398
- joint rr_knee: limit lower=-2.1817 upper=2.1817 effort=2.0 velocity=8.0 -> lower=-1.2217 upper=1.2217 effort=2.0 velocity=8.0; origin xyz=0.000000 0.000000 -0.085000 -> xyz=0.000000 0.000000 -0.070000
- joint rr_pitch: limit lower=-1.7453 upper=1.7453 effort=2.0 velocity=8.0 -> lower=-1.5708 upper=1.5708 effort=2.0 velocity=8.0; origin xyz=-0.100000 0.027200 -0.002000 -> xyz=-0.082650 0.027200 0.000000
- joint rr_splay: limit lower=-0.9599 upper=0.9599 effort=2.0 velocity=8.0 -> lower=-0.7854 upper=0.7854 effort=2.0 velocity=8.0; origin xyz=0.000000 -0.027200 0.012000 -> xyz=0.000000 -0.027200 0.010398
